File: Electronic Design/SAO Core4 V0.1 (KiCAD 8)/SAO_Core4.kicad_sch (KiCad schematic)
At the start: 94 parts, among them Q1 MMBT4403LT1G, Q13 MMBT4403LT1G, Q14 MMBT4401LT1G, Q17 MMBT4403LT1G, Q18 MMBT4401LT1G, Q2 MMBT4401LT1G, Q22 SL3401A, Q3 MMBT4403LT1G, Q4 MMBT4401LT1G, Q5 MMBT4403LT1G, Q6 MMBT4401LT1G, Q7 Q_NMOS_DGS_AO3400A, U1 MCP23017_SS, U10 SN74HC02DR, U7 SSP9193-33M5R, U9 LM393, X1 SAO_conn_SFH11-NBPC-D03-ST-BK, X2 SAO_conn_SFH11-NBPC-D03-ST-BK, X9 QWIIC

Commit message: Refine
Cleanup schematic, plan drive scheme, commit to CM_EN, spare IO.
Parts:
- removed JP3: CME_BYPASS, Jumper:SolderJumper-2_P1.3mm_Bridged_RoundedPad1.0x1.5mm, symbol Jumper:SolderJumper_2_Bridged
- removed JP5: EN_LED1, Jumper:SolderJumper-2_P1.3mm_Open_Pad1.0x1.5mm, symbol Jumper:SolderJumper_2_Open
- removed JP6: EN_GPIO1, Jumper:SolderJumper-2_P1.3mm_Open_Pad1.0x1.5mm, symbol Jumper:SolderJumper_2_Open
- removed R11, R12, R15, R16, R19, R20, R22, R23, R24, R26: 10K, Resistor_SMD:R_0805_2012Metric, symbol Device:R
- added J1: ALT. BATT., Connector_PinSocket_2.54mm:PinSocket_1x02_P2.54mm_Vertical, symbol Connector_Generic:Conn_01x02
- added JP11: CM_SNS_SEL, Jumper:SolderJumper-3_P1.3mm_Bridged12_Pad1.0x1.5mm, symbol Jumper:SolderJumper_3_Bridged12
- added TP6: GPB6, Andy_Footprint_Library:TestPoint_THTPad_D1.5mm_Drill1.0mm, symbol Connector:TestPoint_Probe
- added TP7: GPB7, Andy_Footprint_Library:TestPoint_THTPad_D1.5mm_Drill1.0mm, symbol Connector:TestPoint_Probe
Connections:
- net CM_EN: now also U1.27 (GPA6)
- net GND: now also J1.2 (Pin_2)
- net GPIO1: now also JP11.1 (A)
- net LED_1: now also U1.3 (GPB2); no longer U1.5 (GPB4)
- net LED_2: now also U1.4 (GPB3); no longer U1.6 (GPB5)
- net LED_3: now also U1.5 (GPB4); no longer U1.7 (GPB6)
- net LED_4: now also U1.6 (GPB5); no longer U1.8 (GPB7)
- net VIN: now also J1.1 (Pin_1)
- net CM_Q7N renamed CM_Q7N_9P
- net CM_Q7N_9P: now also R17.2
- net CM_Q7P renamed CM_Q7P_9N
- net CM_Q7P_9N: now also R18.2
- removed net CM_Q9N: R18.2, U1.3 (GPB2)
- removed net CM_Q9P: R17.2, U1.4 (GPB3)
- net CM_SENSE_PULSE renamed CM_SNS_PLS
- net CM_SNS_PLS: now also JP11.2 (C); no longer U1.27 (GPA6)
- net CM_SENSE_RESET renamed CM_SNS_RST
- new net SPARE_GPB6: JP11.3 (B), TP6.1, U1.7 (GPB6)
- new net SPARE_GPB7: TP7.1, U1.8 (GPB7)
Other:
- note added: "GPIO EXPANDER"
- note added: "Review component #ing to match Core16/64/c"
- note added: "Should switching be on low side like adafruit IO expander?"
- note added: "Write Drive Sequence (with sense read always along for the ride): ROW Port: Set ROW transistor current right/left. COL Port: Set CM_EN LOW, CM_SNS_RST HIGH, column transistor current up/down. COL Port: Set CM_EN HIGH, CM_SNS_RST LOW. DELAY as needed COL Port: Set CM_EN CM_EN LOW GPIO 1 (or COL Port B2): Read CM_SNS_PLS and store to SENSE FLAG"
- title: Core4 SAO -> SAO Core4
- moved on the sheet: C10, C11, C12, C13, C14, C15, C19, C2, JP1, JP17, JP18, JP2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

Commit message: Refine schematic
Parts:
- removed J1: ALT. BATT., Connector_PinSocket_2.54mm:PinSocket_1x02_P2.54mm_Vertical, symbol Connector_Generic:Conn_01x02
- removed JP18: CM_CUR_MON, Jumper:SolderJumper-2_P1.3mm_Bridged_RoundedPad1.0x1.5mm, symbol Jumper:SolderJumper_2_Bridged
- R32: renamed from R29; LCSC C17802 -> C17477
- R33: renamed from R30; LCSC C17802 -> C17477
- R44: renamed from R33; value 10K -> 4K7; LCSC C269724 -> C17673
- R60: renamed from R7; value 470 -> 120; LCSC C17710 -> C17437
- R61: renamed from R8; value 470 -> 120; LCSC C17710 -> C17437
- R62: renamed from R9; value 470 -> 120; LCSC C17710 -> C17437
- R63: renamed from R10; value 470 -> 120; LCSC C17710 -> C17437
- renumbered JP11 to JP21, JP10 to JP22, JP2 to JP23, JP4 to JP24, JP1 to JP3, JP7 to JP30, JP8 to JP31, JP9 to JP32, Q7 to Q21, R28 to R27, R27 to R28, R31 to R30, R32 to R31, U1 to U11
Connections:
- net VIN: now also JP22.3 (B); no longer JP22.1 (A)
- net VMEM: now also C12.1, C13.1, C14.1, C15.1, C17.1, C18.1, C19.1, C2.1, JP17.1 (A), JP17.2 (B), JP22.1 (A), JP30.1 (A), JP31.1 (A), JP32.1 (A), R30.1, R31.1, R48.1, R51.1, R54.1, R55.1, U10.14 (VCC), U11.18 (~{RESET}), U11.9 (VDD), U7.5 (OUT), U9.8 (V+)
- removed net 3V3: C12.1, C13.1, C14.1, C15.1, C17.1, C18.1, C19.1, C2.1, JP17.1 (A), JP17.2 (B), JP22.3 (B), JP30.1 (A), JP31.1 (A), JP32.1 (A), R30.1, R31.1, R48.1, R51.1, R54.1, R55.1, U10.14 (VCC), U11.18 (~{RESET}), U11.9 (VDD), U7.5 (OUT), U9.8 (V+)
- net CM_Q1N renamed CMDQ1N
- net CM_Q1P renamed CMDQ1P
- net CM_Q2N renamed CMDQ2N
- net CM_Q2P renamed CMDQ2P
- net CM_Q3N renamed CMDQ3N
- net CM_Q3P renamed CMDQ3P
- net CM_Q7N_9P renamed CMDQ7N9P
- net CM_Q7P_9N renamed CMDQ7P9N
Other:
- note added: "Write Drive Sequence (with sense read always along for the ride): ROW Port: Set ROW transistor left. COL Port: Set CM_EN LOW, CM_SNS_RST HIGH, transistor up/down. COL Port: Set CM_EN HIGH, CM_SNS_RST LOW. DELAY as needed GPIO 1 (or COL Port B2): Read CM_SNS_PLS and store to SENSE data COL Port: Set CM_EN CM_EN LOW"
- note removed: "Review component #ing to match Core16/64/c"
- note removed: "Should switching be on low side like adafruit IO expander?"
- note removed: "Write Drive Sequence (with sense read always along for the ride): ROW Port: Set ROW transistor current right/left. COL Port: Set CM_EN LOW, CM_SNS_RST HIGH, column transistor current up/down. COL Port: Set CM_EN HIGH, CM_SNS_RST LOW. DELAY as needed COL Port: Set CM_EN CM_EN LOW GPIO 1 (or COL Port B2): Read CM_SNS_PLS and store to SENSE FLAG"
- moved on the sheet: JP22
