File: Electronic Design/SAO_Core4_V0.1 Design Files KiCAD 8/SAO_Core4.kicad_pcb (KiCad board)
At the start: 2 copper layers, 50.8 x 63.5 mm, 92 parts, among them Q1 MMBT4403LT1G, Q13 MMBT4403LT1G, Q14 MMBT4401LT1G, Q17 MMBT4403LT1G, Q18 MMBT4401LT1G, Q2 MMBT4401LT1G, Q21 Q_NMOS_DGS_AO3400A, Q22 SL3401A, Q3 MMBT4403LT1G, Q4 MMBT4401LT1G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

Commit message: HWV0.1 as prototyped
Design as released, files organized.
Parts:
- removed R25: 8R2-5%, Resistor_SMD:R_0805_2012Metric
- removed kibuzzard-64178EA5: G***, kibuzzard-64178EA5
- removed kibuzzard-64179D69: G***, kibuzzard-64179D69
- removed kibuzzard-66BD78BD: G***, kibuzzard-66BD78BD
- added JP25: CM_SNS_SEL, Jumper:SolderJumper-3_P1.3mm_Bridged12_Pad1.0x1.5mm, B.Cu at (84.9, 109.4)
- added R7: 8R2-5%, Resistor_SMD:R_0805_2012Metric, B.Cu at (94.6, 130.3)
- added kibuzzard-66C5FD34: G***, kibuzzard-66C5FD34, B.Cu at (85.4, 101.0)
- added kibuzzard-66C5FD67: G***, kibuzzard-66C5FD67, B.Cu at (86.6, 96.6)
- D1, D2, D3, D4: footprint LED_SMD:LED_1206_3216Metric_ReverseMount_Hole1.8x2.4mm -> Andy_Footprint_Library:LED_1206_3216Metric_RevMnt_Hole1.8x2.4mm_custom
- Q22: footprint Package_TO_SOT_SMD:SOT-23-3 -> digikey-footprints:SOT-23-3
- TP20, TP21, TP22, TP23: footprint Andy_Footprint_Library:TestPoint_THTPad_D1.5mm_Drill1.0mm -> TestPoint:TestPoint_Pad_1.5x1.5mm
- kibuzzard-64178DE8, kibuzzard-64178DF4, kibuzzard-64178E7C: moved to B.Cu
- moved kibuzzard-64178DF4 81.9 mm to (98.1, 113.1), turned to 180 degrees
- moved TP22 79.6 mm to (130.4, 130.9)
- moved TP23 76.2 mm to (122.8, 130.9)
- moved R51 71.2 mm to (122.8, 120.4), turned to 0 degrees
- moved R54 70.5 mm to (121.5, 137.5), turned to 0 degrees
- moved R55 70.4 mm to (121.5, 141.0), turned to 0 degrees
- moved C17 69.4 mm to (121.7, 123.7)
- moved C18 69.4 mm to (121.7, 127.2)
- moved R52 68.7 mm to (126.4, 120.4), turned to 0 degrees
- moved R48 68.4 mm to (122.8, 117.1), turned to 0 degrees
- moved TP20 67.5 mm to (122.8, 113.1)
- moved R53 66.3 mm to (130.1, 120.4), turned to 0 degrees
- moved C19 65.9 mm to (125.2, 134.6), turned to 90 degrees
- moved TP21 64.9 mm to (130.4, 113.1)
- moved R49 64.8 mm to (126.4, 117.1), turned to 0 degrees
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- renumbered JP22 to JP21, JP24 to JP22, JP21 to JP24
Connections:
- net /CMDQ1N renamed /CMDQ-1N
- net /CMDQ1P renamed /CMDQ-1P
- net /CMDQ2N renamed /CMDQ-2N
- net /CMDQ2P renamed /CMDQ-2P
- net /CMDQ3N renamed /CMDQ-3N
- net /CMDQ3P renamed /CMDQ-3P
- net /CMDQ7N9P renamed /CMDQ-7N9P
- net /CMDQ7P9N renamed /CMDQ-7P9N
- C12 pad 1: 3V3 -> /3V3_LDO
- JP17 pad 1: 3V3 -> /3V3_LDO
- JP24 pad 1: /GPIO1 -> /GPIO2
- Q17 pad 3: /YL1 -> Net-(Q17-C)
- Q18 pad 3: /YL1 -> Net-(Q17-C)
- U11 pad 27: /CM_EN -> /SPARE_GPA6
- U7 pad 5: 3V3 -> /3V3_LDO
Routing:
- net GND: track 106.9 -> 307.5 mm, vias 0 -> 14
- net 3V3: track 215.2 -> 327.6 mm, vias 4 -> 17
- net /CMDQ-3P: track 0.00 -> 55.3 mm
- net /CM_SENSE_1_IN: track 0.00 -> 54.0 mm, vias 0 -> 2
- net /CMDQ-3N: track 0.00 -> 50.6 mm
- net /CM_SNS_RST: track 0.00 -> 44.2 mm, vias 0 -> 2
- net Net-(Q22-S): track 0.00 -> 42.7 mm
- net /CM_SENSE_2_IN: track 0.00 -> 42.1 mm
- net /LED_2: track 0.00 -> 41.0 mm, vias 0 -> 2
- net /CMDQ-2P: track 0.00 -> 40.8 mm, vias 0 -> 2
- net /SPARE_GPB6: track 0.00 -> 40.0 mm, vias 0 -> 1
- net /CMDQ-2N: track 0.00 -> 40.0 mm, vias 0 -> 2
- net /LED_4: track 0.00 -> 37.6 mm, vias 0 -> 2
- net /SPARE_GPB7: track 0.00 -> 35.7 mm, vias 0 -> 2
- net GMEM: track 53.4 -> 87.5 mm, vias 1 -> 8
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Other:
- rule pad_to_mask_clearance: 0.051 -> 0
- rule solder_mask_min_width: 0.25 -> 0.1016
- board text added: "2GPIO1"
- board text added: "3V3"
- board text added: "3V3 CUR MON"
- board text added: "GMEM CUR MON"
- board text added: "GPA6"
- board text added: "GPB6"
- board text added: "GPB7"
- board text added: "GPIO1"
- board text added: "LOGIC LEVELS 3.3V"
- board text added: "OUT"
- board text added: "PCB: 612-001 REV: 0.1 PCBA: 612-000"
- board text added: "S1"
- board text added: "S2"
- board text added: "S2>IN<S1"
- board text added: "SENSE"
- board text added: "VIN"
- board text removed: "3V3_CUR_MON"
- board text removed: "5VM"
- board text removed: "ALL LOGIC LEVELS 3.3V"
- board text removed: "BACK SIDE"
- board text removed: "BC0_MON"
- board text removed: "BVM"
- board text removed: "CM_CUR_MON"
- board text removed: "DESC: Core64 Logic Board PCB P/N: 112-001 REV: 0.9 (2024-01-25) PCBA P/N: 112-000"
- board text removed: "FRONT SIDE"
- board text removed: "GMEM"
- board text removed: "GND"
- board text removed: "Interactive Core Memory"
- board text removed: "LOGIC BOARD LEVELS 3.3V"
- board text removed: "LR0_MON"
- board text removed: "More information at www.Core64.io"
- board text removed: "Q1-10"
- board text removed: "Q11-20"
- board text removed: "R1- 20"
- board text removed: "RR0_MON"
- board text removed: "S1<OUT>S2"
- board text removed: "S1>IN<S2"
- board text removed: "SYS CUR MON"
- board text removed: "VBUS-VUSB_TIE"
- board text removed: "VMEM"
- board text removed: "VOLTAGE: 3.0-5.5V"
- board text removed: "XB0-3"
- board text removed: "XT0,4:1,5:2,6:3,7"
- board text removed: "YL0-3"
- board text removed: "YL4,6:5,7"
