File: Electronic Design/SAO_Core4_V0.1 Design Files KiCAD 8/SAO_Core4.kicad_sch (KiCad schematic)
At the start: 83 parts, among them Q1 MMBT4403LT1G, Q13 MMBT4403LT1G, Q14 MMBT4401LT1G, Q17 MMBT4403LT1G, Q18 MMBT4401LT1G, Q2 MMBT4401LT1G, Q21 Q_NMOS_DGS_AO3400A, Q22 SL3401A, Q3 MMBT4403LT1G, Q4 MMBT4401LT1G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

Commit message: HWV0.1 as prototyped
Design as released, files organized.
Parts:
- removed R25: 8R2-5%, Resistor_SMD:R_0805_2012Metric, symbol Device:R
- added JP25: CM_SNS_SEL, Jumper:SolderJumper-3_P1.3mm_Bridged12_Pad1.0x1.5mm, symbol Jumper:SolderJumper_3_Bridged12
- added R7: 8R2-5%, Resistor_SMD:R_0805_2012Metric, symbol Device:R
- D1, D2, D3, D4: footprint LED_SMD:LED_1206_3216Metric_ReverseMount_Hole1.8x2.4mm -> Andy_Footprint_Library:LED_1206_3216Metric_RevMnt_Hole1.8x2.4mm_custom
- Q22: footprint Package_TO_SOT_SMD:SOT-23-3 -> digikey-footprints:SOT-23-3
- R21: LCSC C17774 -> C17830
- TP20, TP21, TP22, TP23: footprint Andy_Footprint_Library:TestPoint_THTPad_D1.5mm_Drill1.0mm -> TestPoint:TestPoint_Pad_1.5x1.5mm
- U9: LCSC (none) -> C7955
- renumbered JP22 to JP21, JP24 to JP22, JP21 to JP24
Connections:
- net CM_EN: now also JP25.2 (C); no longer U11.27 (GPA6)
- net GPIO1: now also JP25.1 (A); no longer JP24.1 (A)
- net GPIO2: now also JP24.1 (A)
- net VMEM: no longer C12.1, JP17.1 (A), U7.5 (OUT)
- net YL1: now also R7.1; no longer Q17.3 (C), Q18.3 (C)
- net CMDQ1N renamed CMDQ-1N
- net CMDQ1P renamed CMDQ-1P
- net CMDQ2N renamed CMDQ-2N
- net CMDQ2P renamed CMDQ-2P
- net CMDQ3N renamed CMDQ-3N
- net CMDQ3P renamed CMDQ-3P
- net CMDQ7N9P renamed CMDQ-7N9P
- net CMDQ7P9N renamed CMDQ-7P9N
- new net: Q17.3 (C), Q18.3 (C), R7.2
- new net 3V3_LDO: C12.1, JP17.1 (A), U7.5 (OUT)
- new net SPARE_GPA6: JP25.3 (B), U11.27 (GPA6)
Other:
- moved on the sheet: JP24
