File: Electronic Design/SAO_Core4_V0.2 Design Files KiCAD 8/SAO_Core4.kicad_sch (KiCad schematic)
At the start: 89 parts, among them Q1 MMBT4403LT1G, Q13 MMBT4403LT1G, Q14 MMBT4401LT1G, Q17 MMBT4403LT1G, Q18 MMBT4401LT1G, Q2 MMBT4401LT1G, Q21 Q_NMOS_DGS_AO3400A, Q22 SL3401A, Q3 MMBT4403LT1G, Q4 MMBT4401LT1G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

Commit message: Add SAo Core4 V0.2 files, demo code update
Parts:
- removed C1, C3, C4, C5: 0.1uF, Capacitor_SMD:C_0805_2012Metric, symbol Device:C
- removed L3: Core_64_M-+S_Buttons_4mm, Core_64_KiCad_Library:Core64-M_-_+_S_Buttons, symbol CORE_64_LIBRARY:Core_64_M-+S_Buttons_4mm
- removed Q22: SL3401A, digikey-footprints:SOT-23-3, symbol Device:Q_PMOS_GSD
- removed R10, R11, R8, R9: 10K, Resistor_SMD:R_0805_2012Metric, symbol Device:R_Small
- removed R32, R33: 0, Resistor_SMD:R_0805_2012Metric, symbol Device:R
- removed R44: 4K7, Resistor_SMD:R_0805_2012Metric, symbol Device:R
- removed TP20: S1 IN, TestPoint:TestPoint_Pad_1.5x1.5mm, symbol Connector:TestPoint_Probe
- removed TP21: S2 IN, TestPoint:TestPoint_Pad_1.5x1.5mm, symbol Connector:TestPoint_Probe
- removed TP22: S2 OUT, TestPoint:TestPoint_Pad_1.5x1.5mm, symbol Connector:TestPoint_Probe
- removed TP23: S1 OUT, TestPoint:TestPoint_Pad_1.5x1.5mm, symbol Connector:TestPoint_Probe
- removed U1: SI7210-B-00-IV, Package_TO_SOT_SMD:SOT-23-5, symbol Core64-CB-v0.6-rescue:SI7210-Sensor_Magnetic
- removed U2: SI7210-B-02-IV, Package_TO_SOT_SMD:SOT-23-5, symbol Core64-CB-v0.6-rescue:SI7210-Sensor_Magnetic
- removed U3: SI7210-B-03-IV, Package_TO_SOT_SMD:SOT-23-5, symbol Core64-CB-v0.6-rescue:SI7210-Sensor_Magnetic
- removed U4: SI7210-B-04-IV, Package_TO_SOT_SMD:SOT-23-5, symbol Core64-CB-v0.6-rescue:SI7210-Sensor_Magnetic
- added J1: V+ALT, Connector_PinSocket_1.27mm:PinSocket_1x01_P1.27mm_Vertical, symbol Connector_Generic:Conn_01x01
- added JP1: VSEL, Jumper:SolderJumper-3_P1.3mm_Bridged12_Pad1.0x1.5mm, symbol Jumper:SolderJumper_3_Bridged12
- R21, R7: value 8R2-5% -> 6R8-5%; LCSC C17830 -> C17774
- R27: value 4K7 -> 10K; LCSC C17673 -> C17414
- R30, R31: value 1K2 -> 10K; Insert (none) -> YES; LCSC C17379 -> C17414; Populate no -> (none); Value_Modifier (none) -> 10%
- R54, R55: value 1K2 -> 10K; Insert (none) -> YES; Insert? Yes -> (none); LCSC C17379 -> C17414; Populate yes -> (none)
- SW1: footprint SMD4_SW_EVQP7J_PAN -> Andy_Footprint_Library:SMD4_SW_EVQP7J_PAN; LCSC (none) -> C2828254
- U10: LCSC C350559 -> C6809
- X1: footprint Andy_Footprint_Library:Badgelife-SAOv169-BADGE-2x3 -> Andy_Footprint_Library:Badgelife-SAOv169-BADGE-2x3-Edge-Connect-no-front-text
- renumbered R60 to R61, R61 to R62, R62 to R63, R63 to R64
Connections:
- net I2C_SCL is gone; now on net SCL: R30.2, U11.12 (SCK)
- net I2C_SDA is gone; now on net SDA: R31.2, U11.13 (SDA)
- net CMDQ-7N: now also U11.5 (GPB4); no longer U11.1 (GPB0)
- net CMDQ-7P: now also U11.6 (GPB5); no longer U11.2 (GPB1)
- net GND: now also SW1.3, SW1.4
- net GPIO1: now also SW1.1, SW1.2
- net LED_1: now also U11.1 (GPB0); no longer U11.3 (GPB2)
- net LED_2: now also U11.2 (GPB1); no longer U11.4 (GPB3)
- net LED_3: now also U11.3 (GPB2); no longer U11.5 (GPB4)
- net LED_4: now also U11.4 (GPB3); no longer U11.6 (GPB5)
- net VIN: now also JP1.1 (A)
- net XT0,1: no longer Q5.3 (C), Q6.3 (C), R21.1
- net at C10.1, U7.1 (IN), U7.3 (EN): now also JP1.2 (C)
- new net: Q5.3 (C), Q6.3 (C), R21.1
- new net: J1.1 (Pin_1), JP1.3 (B)
Other:
- note added: "I2C PULLUPS"
- note added: "MODE BUTTON"
- note added: "Write Drive Sequence (with sense read always along for the ride): ROW Port: Set ROW transistors enabled as needed. COL Port: Set CM_EN LOW, CM_SNS_RST HIGH, COL transistors disabled. COL Port: Set CM_EN HIGH, CM_SNS_RST LOW, COL transistors as needed. GPIO 1: Read CM_SNS_PLS and store to SENSE data array. COL Port: Set CM_EN CM_EN LOW, CM_SNS_RST LOW, COL transistors disabled."
- note removed: "DIGITAL LOGIC GROUND"
- note removed: "HALL SENSORS"
- note removed: "I2C BUFFER"
- note removed: "I2C configurable hall sensors, not just a switch. Silicon Labs SI7210-B-xx-IV (00, 02, 03, 04) Low (push-pull) up to 20 mT, SOT23-5 Recommended sensitivity ± (N and S) 3-7 mT (30-70 Gauss)"
- note removed: "P-CHNL"
- note removed: "REVERSE POLARITY PROTECTION"
- note removed: "RPP"
- note removed: "Rds(on)0.06"
- note removed: "SILKSCREEN: 0x30"
- note removed: "SILKSCREEN: 0x31"
- note removed: "SILKSCREEN: 0x32"
- note removed: "SILKSCREEN: 0x33"
- note removed: "TODO: Shift LED connections up 2 pins, tying B3/4 to 7N/7P. The order will look cleaner, and LED pixel numbering will match GPB numbers."
- note removed: "WIP"
- note removed: "Write Drive Sequence (with sense read always along for the ride): ROW Port: Set ROW transistor left. COL Port: Set CM_EN LOW, CM_SNS_RST HIGH, transistor up/down. COL Port: Set CM_EN HIGH, CM_SNS_RST LOW. DELAY as needed GPIO 1 (or COL Port B2): Read CM_SNS_PLS and store to SENSE data COL Port: Set CM_EN CM_EN LOW"
- moved on the sheet: JP3, Q21, R27, R28, SW1
